Commit message: update xacro sensors

File: description/gps.xacro (robot description, xacro)
@@ -1,23 +1,40 @@
 <?xml version="1.0"?>
-<robot xmlns:xacro="http://www.ros.org/wiki/xacro">
-  <joint name="gps_joint" type="fixed">
-    <parent link="chassis"/>
-    <child link="gps_link"/>
-    <origin xyz="0.1675 0.035 0.144" rpy="0 0 0"/>
-  </joint>
-  <link name="gps_link">
-    <visual>
-      <geometry>
-        <box size="0.03 0.03 0.01"/>
-      </geometry>
-      <material name="black"/>
-    </visual>
-  </link>
-  <gazebo reference="gps_link">
-    <sensor name="navsat_sensor" type="navsat">
-      <always_on>true</always_on>
-      <update_rate>30</update_rate>
-      <topic>/gps</topic>
-    </sensor>
-  </gazebo>
+<robot xmlns:xacro="http://www.ros.org/wiki/xacro" >
+    <joint name="gps_joint" type="fixed">
+        <parent link="chassis"/>
+        <child link="gps_link"/>
+        <origin xyz="0.1675 0.035 0.144" rpy="0 0 0"/>
+    </joint>
+    <link name="gps_link">
+        <visual>
+            <geometry>
+                <box size="0.03 0.03 0.01"/>
+            </geometry>
+            <material name="black"/>
+        </visual>
+    </link>
+    <gazebo reference="gps_link">
+      <selfCollide>false</selfCollide>
+    </gazebo>
+    <gazebo reference="gps_link">
+        <material>Gazebo/Red</material>
+        <sensor name="gps_sensor" type="navsat">
+        <topic>/nav_msgs</topic>
+        <update_rate>5</update_rate>
+        <navsat>
+            <reference_latitude>-25.330480</reference_latitude>
+            <reference_longitude>-57.518124</reference_longitude>
+            <reference_altitude>80.0</reference_altitude>
+            <velocity_smoothing>true</velocity_smoothing>
+            <noise type="gaussian">
+                <mean>0.0</mean>
+                <stddev>0.00001</stddev>
+            </noise>
+        </navsat>
+        <plugin
+            filename="gz-sim-navsat-system"
+            name="gz::sim::systems::NavSat">
+        </plugin>
+        </sensor>
+    </gazebo>
 </robot>
