Commit message: update name

File: description/ros2_control.xacro (robot description, xacro)
@@ -56,6 +56,6 @@
     <gazebo>
         <plugin name="gz_ros2_control::GazeboSimROS2ControlPlugin" filename="libgz_ros2_control-system.so">
-            <parameters>$(find hexapot_pkg)/config/my_controllers.yaml</parameters>
-            <parameters>$(find hexapot_pkg)/config/gaz_ros2_ctl_use_sim.yaml</parameters>
+            <parameters>$(find hexapod_pkg)/config/my_controllers.yaml</parameters>
+            <parameters>$(find hexapod_pkg)/config/gaz_ros2_ctl_use_sim.yaml</parameters>
         </plugin>
     </gazebo>

File: description_hexapod/base_uttu.urdf.xacro (robot description, xacro)
@@ -12,5 +12,5 @@
           <origin xyz="0 0 0" rpy="0 0 0" />
           <geometry>
-            <mesh filename="$(find hexapot_pkg)/meshes/body.STL"  scale="1 1 1"/>
+            <mesh filename="$(find hexapod_pkg)/meshes/body.STL"  scale="1 1 1"/>
           </geometry>
           <material name="Grey">
@@ -20,5 +20,5 @@
 	  <collision>
 		<geometry>
-		  <mesh filename="$(find hexapot_pkg)/meshes/body_coll.STL"/>
+		  <mesh filename="$(find hexapod_pkg)/meshes/body_coll.STL"/>
 		</geometry>
 	  </collision>

File: description_hexapod/hexapod_robot_gazebo.xacro (robot description, xacro)
@@ -5,5 +5,5 @@
     <gazebo>
       <plugin filename="libgz_ros2_control-system.so" name="gz_ros2_control::GazeboSimROS2ControlPlugin">
-        <parameters>$(find hexapot_pkg)/config/my_hexapod_controllers.yaml</parameters>
+        <parameters>$(find hexapod_pkg)/config/my_hexapod_controllers.yaml</parameters>
       </plugin>
     </gazebo>

File: description_hexapod/holder_pi_hexapod.xacro (robot description, xacro)
@@ -10,5 +10,5 @@
           <origin xyz="0 0 0" rpy="0 0 0" />
           <geometry>
-            <mesh filename="$(find hexapot_pkg)/meshes/holder_pi_uttu.STL"  scale="0.0012 0.0012 0.0012"/>
+            <mesh filename="$(find hexapod_pkg)/meshes/holder_pi_uttu.STL"  scale="0.0012 0.0012 0.0012"/>
           </geometry>
           <material name="Grey">

File: description_hexapod/legs_uttu.urdf.xacro (robot description, xacro)
@@ -30,5 +30,5 @@
         <origin xyz="0 -0.0252 0"/>
         <geometry>
-          <mesh filename="$(find hexapot_pkg)/meshes/connect.STL"/>
+          <mesh filename="$(find hexapod_pkg)/meshes/connect.STL"/>
         </geometry>
           <material name="Blue">
@@ -39,5 +39,5 @@
         <origin xyz="0 -${connect_offset} 0"/>
         <geometry>
-          <mesh filename="$(find hexapot_pkg)/meshes/connect_coll.STL"/>
+          <mesh filename="$(find hexapod_pkg)/meshes/connect_coll.STL"/>
         </geometry>
       </collision>
@@ -63,5 +63,5 @@
       <origin xyz="0 -0.0252 0"/>
       <geometry>
-        <mesh filename="$(find hexapot_pkg)/meshes/connect.STL"/>
+        <mesh filename="$(find hexapod_pkg)/meshes/connect.STL"/>
       </geometry>
           <material name="Blue">
@@ -72,5 +72,5 @@
         <origin xyz="0 -${connect_offset} 0"/>
         <geometry>
-          <mesh filename="$(find hexapot_pkg)/meshes/connect_coll.STL"/>
+          <mesh filename="$(find hexapod_pkg)/meshes/connect_coll.STL"/>
         </geometry>
       </collision>
@@ -98,5 +98,5 @@
         <origin xyz="0 0 0"/>
         <geometry>
-          <mesh filename="$(find hexapot_pkg)/meshes/thigh_l.STL"/>
+          <mesh filename="$(find hexapod_pkg)/meshes/thigh_l.STL"/>
         </geometry>
           <material name="Grey">
@@ -107,5 +107,5 @@
         <origin xyz="0 0 0"/>
         <geometry>
-          <mesh filename="$(find hexapot_pkg)/meshes/thigh_l_coll.STL"/>
+          <mesh filename="$(find hexapod_pkg)/meshes/thigh_l_coll.STL"/>
         </geometry>
       </collision>
@@ -133,5 +133,5 @@
         <origin xyz="0 0 0"/>
         <geometry>
-          <mesh filename="$(find hexapot_pkg)/meshes/tibia_l.STL"/>
+          <mesh filename="$(find hexapod_pkg)/meshes/tibia_l.STL"/>
         </geometry>
           <material name="Blue">
@@ -142,5 +142,5 @@
         <origin xyz="0 0 0"/>
         <geometry>
-          <mesh filename="$(find hexapot_pkg)/meshes/tibia_l_coll.STL"/>
+          <mesh filename="$(find hexapod_pkg)/meshes/tibia_l_coll.STL"/>
         </geometry>
       </collision>
